Commit message: added docker-compose and urdf fixes
Signed-off-by: Sezgin Atabas <atabassezgin@gmail.com>

File: ros2/drone_vision_pkg/urdf/drone_description.urdf.xacro (robot description, xacro)
@@ -1,18 +1,21 @@
-<robot name="drone" xmlns:xacro="http://ros.org/wiki/xacro">
+<robot name="stereolabs_camera" xmlns:xacro="http://ros.org/wiki/xacro">
   <xacro:arg name="camera_name"   default="zed" />
-  <xacro:arg name="camera_model"  default="zedm" />
-  <xacro:arg name="use_zed_localization" default="true" />
-  <!-- Include the robot  -->
-  <xacro:include filename="$(find drone_vision_pkg)/urdf/drone_body.xacro" />
-  <!-- Add one ZED Camera -->
-  <xacro:include filename="$(find zed_wrapper)/urdf/zed_macro.urdf.xacro" />@
-  <xacro:zed_camera name="$(arg camera_name)" model="$(arg camera_model)" />
-  <joint name="$(arg camera_name)_joint" type="fixed">
-      <parent link="base_link"/>
-      <child link="$(arg camera_name)_camera_link"/>
-      <origin
-        xyz="0.12 0.0 0.08"
-        rpy="0 0 0"
-      />
-  </joint>
+  <xacro:arg name="camera_model"  default="zed" />
+  <xacro:arg name="custom_baseline"  default="0.0" />
+  <!-- If GNSS fusion is enabled the position of the antenna with respect to the camera mount point is required -->
+  <xacro:arg name="enable_gnss"   default="false" />
+  <xacro:arg name="gnss_x" default="0.0" />
+  <xacro:arg name="gnss_y" default="0.0" />
+  <xacro:arg name="gnss_z" default="0.0" />
+  <xacro:include filename="$(find zed_wrapper)/urdf/zed_macro.urdf.xacro" />
+  <xacro:zed_camera name="$(arg camera_name)" model="$(arg camera_model)" custom_baseline="$(arg custom_baseline)" enable_gnss="$(arg enable_gnss)">
+      <joint name="$(arg camera_name)_joint" type="fixed">
+          <parent link="base_link"/>
+          <child link="$(arg camera_name)_camera_link"/>
+          <origin
+            xyz="0.15 0.0 0.06"
+            rpy="0 0 0"
+          />
+      </joint>
+  </xacro:zed_camera>
 </robot>
